File: Hardware/Qwiic_Pocket_Dev_ESP32_C6_Trim/Qwiic_Pocket_Dev_ESP32_C6.kicad_pcb (KiCad board)
At the start: 4 copper layers, 17.2 x 25.4 mm, 55 parts, among them J1 USB Female Type C Connector, J4 QWIIC_RIGHT_ANGLE, Q1 20V/4.2A/52mΩ/1.4W, U1 ESP32-C6-MINI-1, U2 RT9080-33GJ5, U3 MCP73831

Commit message: edges 1
Parts:
- removed FRAME1: FRAME-LETTER, CREATIVE_COMMONS
- removed LOGO1: SFE_LOGO_NAME_FLAMEBLANK, BLANK
- removed U$24: , ORDERING_INSTRUCTIONS
Other:
- board outline removed
- board text removed: "1"
- board text removed: "2"
- board text removed: "3"
- board text removed: "4"
- board text removed: "4-layer JLC7628 Stackup Material: TG135-140 1oz outer layers 0.5oz inner layers Board thickness: 1.6mm Soldermask: Red Silkscreen: White Surface Finish: Lead-Free HASL"
- board text removed: "Dryw Wade"
- board text removed: "v10"
