File: Hardware/ESP32_C6_BME688/BME688_Daughterboard/BME688_Daughterboard.kicad_pcb (KiCad board)
At the start: 2 copper layers, 7.5 x 7.5 mm, 3 parts, among them J4 Carrier_Header, U2 BME688

Commit message: adding perpendicular daughter board to main board's 3d print
Parts:
- J4: footprint Connector_PinHeader_1.27mm:PinHeader_1x04_P1.27mm_Vertical -> Connector_PinHeader_1.27mm:PinHeader_1x04_P1.27mm_Horizontal
