File: Hardware/ESP32_C6_BME688_HYBRID0402/ESP32_C6_BME688_HYBRID0402.kicad_pcb (KiCad board)
At the start: 2 copper layers, 24.5 x 20 mm, 13 parts, among them J1 USB_C, J2 JST_PH_2PIN, J3 Daughterboard_Interface, U1 ESP32-C6-MINI-1, U3 MCP73831, U4 AP2112K-3.3

Commit message: fixed all connection issues
Parts:
- moved R2 10.2 mm to (111.4, 116.4)
- moved J3 2.40 mm to (101.2, 110.8)
- moved U1 2.06 mm to (110.0, 108.0)
- moved R5 1.51 mm to (111.4, 119.0)
- moved J1 0.98 mm to (121.2, 114.7)
Routing:
- net VSYS: track 36.6 -> 23.2 mm, vias 0 -> 2
- net I2C0_SCL: track 5.31 -> 16.3 mm, vias 0 -> 1
- net USB_DP: track 25.5 -> 15.7 mm, vias 2 -> 0
- net CC1: track 14.0 -> 5.03 mm
- net VBAT: track 26.2 -> 33.8 mm, vias 0 -> 4
- net +3V3: track 28.3 -> 33.8 mm, vias 0 -> 3
- net USB_DM: track 25.6 -> 21.3 mm, vias 0 -> 2
- net CC2: track 10.3 -> 12.7 mm
- net VBUS_5V: track 22.1 -> 24.3 mm
- net GND: track 98.2 -> 96.2 mm, vias 1 -> 2
- net I2C0_SDA: track 10.1 -> 11.4 mm, vias 0 -> 1
